Commit message: Fixed Driving problem

File: src/rocker_description/urdf/rocker.urdf.xacro (robot description, xacro)
@@ -151,5 +151,5 @@
   <joint
     name="front_right_wheel_joint"
-    type="revolute">
+    type="continuous">
     <origin
       xyz="-0.00064706 -0.090897 -0.080968"
@@ -165,5 +165,5 @@
       upper="10"
       effort="10"
-      velocity="20" />
+      velocity="100" />
   </joint>
   <!-- Front Left Module -->
@@ -268,5 +268,5 @@
   <joint
     name="front_left_wheel_joint"
-    type="revolute">
+    type="continuous">
     <origin
       xyz="0.0006707 0.090897 -0.080967"
@@ -282,5 +282,5 @@
       upper="10"
       effort="10"
-      velocity="20" />
+      velocity="100" />
   </joint>
   <!-- Rear Right Module -->
@@ -385,5 +385,5 @@
   <joint
     name="rear_right_wheel_joint"
-    type="revolute">
+    type="continuous">
     <origin
       xyz="-0.00064706 -0.090897 -0.080968"
@@ -399,5 +399,5 @@
       upper="10"
       effort="10"
-      velocity="20" />
+      velocity="100" />
   </joint>
   <!-- Rear Left Module -->
@@ -502,5 +502,5 @@
   <joint
     name="rear_left_wheel_joint"
-    type="revolute">
+    type="continuous">
     <origin
       xyz="0.0006707 0.090897 -0.080967"
@@ -516,43 +516,43 @@
       upper="10"
       effort="10"
-      velocity="20" />
-  </joint>
- <!-- === DRIVE WHEEL TRANSMISSIONS (Velocity) === -->
-  <transmission name="front_right_wheel_trans">
-    <type>transmission_interface/SimpleTransmission</type>
-    <joint name="front_right_wheel_joint">
-      <hardwareInterface>hardware_interface/VelocityJointInterface</hardwareInterface>
-    </joint>
-    <actuator name="front_right_wheel_motor">
-      <hardwareInterface>hardware_interface/VelocityJointInterface</hardwareInterface>
-      <mechanicalReduction>1</mechanicalReduction>
-    </actuator>
-  </transmission>
-  <transmission name="front_left_wheel_trans">
-    <type>transmission_interface/SimpleTransmission</type>
-    <joint name="front_left_wheel_joint">
-      <hardwareInterface>hardware_interface/VelocityJointInterface</hardwareInterface>
-    </joint>
-    <actuator name="front_left_wheel_motor">
-      <hardwareInterface>hardware_interface/VelocityJointInterface</hardwareInterface>
-      <mechanicalReduction>1</mechanicalReduction>
-    </actuator>
-  </transmission>
-  <transmission name="rear_right_wheel_trans">
-    <type>transmission_interface/SimpleTransmission</type>
-    <joint name="rear_right_wheel_joint">
-      <hardwareInterface>hardware_interface/VelocityJointInterface</hardwareInterface>
-    </joint>
-    <actuator name="rear_right_wheel_motor">
-      <hardwareInterface>hardware_interface/VelocityJointInterface</hardwareInterface>
-      <mechanicalReduction>1</mechanicalReduction>
-    </actuator>
-  </transmission>
-  <transmission name="rear_left_wheel_trans">
-    <type>transmission_interface/SimpleTransmission</type>
-    <joint name="rear_left_wheel_joint">
-      <hardwareInterface>hardware_interface/VelocityJointInterface</hardwareInterface>
-    </joint>
-    <actuator name="rear_left_wheel_motor">
+      velocity="100" />
+  </joint>
+<!-- === DRIVE WHEEL TRANSMISSIONS (Velocity) === -->
+  <transmission name="front_left_trans">
+    <type>transmission_interface/SimpleTransmission</type>
+    <joint name="front_left_joint">
+      <hardwareInterface>hardware_interface/VelocityJointInterface</hardwareInterface>
+    </joint>
+    <actuator name="front_left_motor">
+      <hardwareInterface>hardware_interface/VelocityJointInterface</hardwareInterface>
+      <mechanicalReduction>1</mechanicalReduction>
+    </actuator>
+  </transmission>
+  <transmission name="rear_left_trans">
+    <type>transmission_interface/SimpleTransmission</type>
+    <joint name="rear_left_joint">
+      <hardwareInterface>hardware_interface/VelocityJointInterface</hardwareInterface>
+    </joint>
+    <actuator name="rear_left_motor">
+      <hardwareInterface>hardware_interface/VelocityJointInterface</hardwareInterface>
+      <mechanicalReduction>1</mechanicalReduction>
+    </actuator>
+  </transmission>
+  <transmission name="front_right_trans">
+    <type>transmission_interface/SimpleTransmission</type>
+    <joint name="front_right_joint">
+      <hardwareInterface>hardware_interface/VelocityJointInterface</hardwareInterface>
+    </joint>
+    <actuator name="front_right_motor">
+      <hardwareInterface>hardware_interface/VelocityJointInterface</hardwareInterface>
+      <mechanicalReduction>1</mechanicalReduction>
+    </actuator>
+  </transmission>
+  <transmission name="rear_right_trans">
+    <type>transmission_interface/SimpleTransmission</type>
+    <joint name="rear_right_joint">
+      <hardwareInterface>hardware_interface/VelocityJointInterface</hardwareInterface>
+    </joint>
+    <actuator name="rear_right_motor">
       <hardwareInterface>hardware_interface/VelocityJointInterface</hardwareInterface>
       <mechanicalReduction>1</mechanicalReduction>

File: src/rocker_description/urdf/rocker_gazebo.xacro (robot description, xacro)
@@ -3,37 +3,37 @@
   <!-- Wheels -->
   <gazebo reference="front_left_wheel">
-    <mu1>1000000000000000.0</mu1>
-    <mu2>1000000000000000.0</mu2>
-    <kp>1000000000000.0</kp>
+    <mu1>1.0</mu1>
+    <mu2>1.0</mu2>
+    <kp>1e6</kp>
     <kd>10.0</kd>
     <minDepth>0.001</minDepth>
-    <maxVel>0.1</maxVel>
+    <maxVel>0.5</maxVel>
     <fdir1>1 0 0</fdir1>
   </gazebo>
   <gazebo reference="rear_right_wheel">
-    <mu1>1000000000000000.0</mu1>
-    <mu2>1000000000000000.0</mu2>
-    <kp>1000000000000.0</kp>
+    <mu1>1.0</mu1>
+    <mu2>1.0</mu2>
+    <kp>1e6</kp>
     <kd>10.0</kd>
     <minDepth>0.001</minDepth>
-    <maxVel>0.1</maxVel>
+    <maxVel>0.5</maxVel>
     <fdir1>1 0 0</fdir1>
   </gazebo>
   <gazebo reference="rear_left_wheel">
-    <mu1>1000000000000000.0</mu1>
-    <mu2>1000000000000000.0</mu2>
-    <kp>1000000000000.0</kp>
+    <mu1>1.0</mu1>
+    <mu2>1.0</mu2>
+    <kp>1e6</kp>
     <kd>10.0</kd>
     <minDepth>0.001</minDepth>
-    <maxVel>0.1</maxVel>
+    <maxVel>0.5</maxVel>
     <fdir1>1 0 0</fdir1>
   </gazebo>
   <gazebo reference="front_right_wheel">
-    <mu1>1000000000000000.0</mu1>
-    <mu2>1000000000000000.0</mu2>
-    <kp>1000000000000.0</kp>
+    <mu1>1.0</mu1>
+    <mu2>1.0</mu2>
+    <kp>1e6</kp>
     <kd>10.0</kd>
     <minDepth>0.001</minDepth>
-    <maxVel>0.1</maxVel>
+    <maxVel>0.5</maxVel>
     <fdir1>1 0 0</fdir1>
   </gazebo>

File: src/rocker_description/urdf/rocker_ros2_control.xacro (robot description, xacro)
@@ -13,6 +13,6 @@
     <joint name="front_right_wheel_joint">
       <command_interface name="velocity">
-        <param name="min">-1</param>
-        <param name="max">1</param>
+        <param name="min">-10</param>
+        <param name="max">10</param>
       </command_interface>
       <state_interface name="position"/>
@@ -21,6 +21,6 @@
     <joint name="front_left_wheel_joint">
       <command_interface name="velocity">
-        <param name="min">-1</param>
-        <param name="max">1</param>
+        <param name="min">-10</param>
+        <param name="max">10</param>
       </command_interface>
       <state_interface name="position"/>
@@ -29,6 +29,6 @@
     <joint name="rear_left_wheel_joint">
       <command_interface name="velocity">
-        <param name="min">-1</param>
-        <param name="max">1</param>
+        <param name="min">-10</param>
+        <param name="max">10</param>
       </command_interface>
       <state_interface name="position"/>
@@ -37,6 +37,6 @@
     <joint name="rear_right_wheel_joint">
       <command_interface name="velocity">
-        <param name="min">-1</param>
-        <param name="max">1</param>
+        <param name="min">-10</param>
+        <param name="max">10</param>
       </command_interface>
       <state_interface name="position"/>

Commit message: First iteration for rocker-Chassis Collapses

File: src/rocker_description/urdf/rocker.urdf.xacro (robot description, xacro)
@@ -14,15 +14,15 @@
     <inertial>
       <origin
-        xyz="0.00050491 -6.865E-06 0.018432"
-        rpy="0 0 0" />
-      <mass
-        value="4.3525" />
-      <inertia
-        ixx="0.012465"
-        ixy="5.2568E-06"
-        ixz="1.0799E-05"
-        iyy="0.012459"
-        iyz="-7.1925E-08"
-        izz="0.022004" />
+        xyz="-0.0029178 -1.0243E-05 0.026001"
+        rpy="0 0 0" />
+      <mass
+        value="3.0355" />
+      <inertia
+        ixx="0.011434"
+        ixy="8.2789E-18"
+        ixz="-1.2087E-05"
+        iyy="0.0094299"
+        iyz="-3.1877E-20"
+        izz="0.018372" />
     </inertial>
     <visual>
@@ -37,5 +37,5 @@
         name="">
         <color
-          rgba="0.75294 0.75294 0.75294 1" />
+          rgba="1 0 0 1" />
       </material>
     </visual>
@@ -50,28 +50,27 @@
     </collision>
   </link>
-  <!-- Front Right Module -->
-  <link
-    name="steer_front_right">
-    <inertial>
-      <origin
-        xyz="-0.000580011325193364 -0.0211614748892629 -0.0742015840408135"
-        rpy="0 0 0" />
-      <mass
-        value="0.0538768865361953" />
-      <inertia
-        ixx="1.72828728418579E-05"
-        ixy="1.86500624352126E-10"
-        ixz="-7.06469401373181E-08"
-        iyy="1.26504994050704E-05"
-        iyz="-2.82990645413841E-12"
-        izz="1.01158709169347E-05" />
-    </inertial>
-    <visual>
-      <origin
-        xyz="0 0 0"
-        rpy="0 0 0" />
-      <geometry>
-        <mesh
-          filename="package://rocker_description/meshes/steer_front_right.STL" />
+  <link
+    name="diff_link">
+    <inertial>
+      <origin
+        xyz="0.0236047033494922 3.38568454466559E-07 0.00680399174365073"
+        rpy="0 0 0" />
+      <mass
+        value="0.218473302594947" />
+      <inertia
+        ixx="0.000709218973632844"
+        ixy="-4.54869495674156E-11"
+        ixz="-5.80923680880486E-07"
+        iyy="2.67923062348123E-05"
+        iyz="-9.28184396595003E-10"
+        izz="0.000717476916941679" />
+    </inertial>
+    <visual>
+      <origin
+        xyz="0 0 0"
+        rpy="0 0 0" />
+      <geometry>
+        <mesh
+          filename="package://rocker_description/meshes/diff_link.STL" />
       </geometry>
       <material
@@ -87,40 +86,156 @@
       <geometry>
         <mesh
-          filename="package://rocker_description/meshes/steer_front_right.STL" />
-      </geometry>
-    </collision>
-  </link>
-  <joint
-    name="steer_front_right_joint"
+          filename="package://rocker_description/meshes/diff_link.STL" />
+      </geometry>
+    </collision>
+  </link>
+  <joint
+    name="diff_link_joint"
     type="revolute">
     <origin
-      xyz="0.10649 -0.16648 -0.031065"
+      xyz="0.071998 -1.0243E-05 0.066001"
       rpy="0 0 0" />
     <parent
       link="base_link" />
     <child
-      link="steer_front_right" />
-    <axis
-      xyz="0 0 -1" />
-    <limit
-      lower="-1.57"
-      upper="1.57"
-      effort="2"
-      velocity="3.14" />
-  </joint>
-  <link
-    name="front_right_wheel">
-    <inertial>
-      <origin
-        xyz="1.85114703565858E-08 -1.36100179737308E-09 0.00840874583108253"
+      link="diff_link" />
+    <axis
+      xyz="0 0 -1" />
+    <limit
+      lower="-0.785"
+      upper="0.785"
+      effort="10"
+      velocity="20" />
+  </joint>
+  <link
+    name="T_left">
+    <inertial>
+      <origin
+        xyz="-0.00596279656055823 0.0193116567400055 0.0182177510881137"
+        rpy="0 0 0" />
+      <mass
+        value="0.548279468054" />
+      <inertia
+        ixx="0.000160712183061877"
+        ixy="-1.1829517489236E-05"
+        ixz="4.65340927469138E-08"
+        iyy="0.00145712336718833"
+        iyz="2.38546499162641E-06"
+        izz="0.00150112676275928" />
+    </inertial>
+    <visual>
+      <origin
+        xyz="0 0 0"
+        rpy="0 0 0" />
+      <geometry>
+        <mesh
+          filename="package://rocker_description/meshes/T_left.STL" />
+      </geometry>
+      <material
+        name="">
+        <color
+          rgba="0.752941176470588 0.752941176470588 0.752941176470588 1" />
+      </material>
+    </visual>
+    <collision>
+      <origin
+        xyz="0 0 0"
+        rpy="0 0 0" />
+      <geometry>
+        <mesh
+          filename="package://rocker_description/meshes/T_left.STL" />
+      </geometry>
+    </collision>
+  </link>
+  <joint
+    name="T_left_joint"
+    type="revolute">
+    <origin
+      xyz="-0.0750000000000018 0.129999999999997 -0.0599999999999974"
+      rpy="-1.5707963267949 0 0" />
+    <parent
+      link="diff_link" />
+    <child
+      link="T_left" />
+    <axis
+      xyz="0 0 -1" />
+    <limit
+      lower="-0.785"
+      upper="0.785"
+      effort="10"
+      velocity="20" />
+  </joint>
+  <link
+    name="steer_fl">
+    <inertial>
+      <origin
+        xyz="-0.000138607396474422 0.0211614748792864 -0.0742037212781577"
+        rpy="0 0 0" />
+      <mass
+        value="0.0538768872920871" />
+      <inertia
+        ixx="1.72835692626109E-05"
+        ixy="1.86515416826833E-10"
+        ixz="1.22948666319558E-09"
+        iyy="1.26504997120413E-05"
+        iyz="1.03710843764432E-12"
+        izz="1.01151748078112E-05" />
+    </inertial>
+    <visual>
+      <origin
+        xyz="0 0 0"
+        rpy="0 0 0" />
+      <geometry>
+        <mesh
+          filename="package://rocker_description/meshes/steer_fl.STL" />
+      </geometry>
+      <material
+        name="">
+        <color
+          rgba="0.752941176470588 0.752941176470588 0.752941176470588 1" />
+      </material>
+    </visual>
+    <collision>
+      <origin
+        xyz="0 0 0"
+        rpy="0 0 0" />
+      <geometry>
+        <mesh
+          filename="package://rocker_description/meshes/steer_fl.STL" />
+      </geometry>
+    </collision>
+  </link>
+  <joint
+    name="steer_fl_joint"
+    type="revolute">
+    <origin
+      xyz="0.110151534483122 0.0359863916031299 0.0365656792826139"
+      rpy="1.5707963267949 0 0" />
+    <parent
+      link="T_left" />
+    <child
+      link="steer_fl" />
+    <axis
+      xyz="0 0 -1" />
+    <limit
+      lower="-3.14"
+      upper="3.14"
+      effort="10"
+      velocity="20" />
+  </joint>
+  <link
+    name="fl_wheel">
+    <inertial>
+      <origin
+        xyz="1.69573641517484E-08 -7.54815843162504E-09 -0.00840874583108248"
         rpy="0 0 0" />
       <mass
         value="0.13017290647518" />
       <inertia
-        ixx="0.00012477805886062"
-        ixy="-3.65428145722413E-11"
-        ixz="8.51352948296458E-12"
-        iyy="0.000124777992131831"
-        iyz="-7.24734628585044E-12"
+        ixx="0.000124778074397082"
+        ixy="-7.56745177284866E-12"
+        ixz="-1.0927757268495E-11"
+        iyy="0.000124777976595369"
+        iyz="-2.36402552332323E-12"
         izz="0.000234671292019044" />
     </inertial>
@@ -131,5 +246,5 @@
       <geometry>
         <mesh
-          filename="package://rocker_description/meshes/front_right_wheel.STL" />
+          filename="package://rocker_description/meshes/fl_wheel.STL" />
       </geometry>
       <material
@@ -145,18 +260,18 @@
       <geometry>
         <mesh
-          filename="package://rocker_description/meshes/front_right_wheel.STL" />
-      </geometry>
-    </collision>
-  </link>
-  <joint
-    name="front_right_wheel_joint"
+          filename="package://rocker_description/meshes/fl_wheel.STL" />
+      </geometry>
+    </collision>
+  </link>
+  <joint
+    name="fl_wheel_joint"
     type="continuous">
     <origin
-      xyz="-0.00064706 -0.090897 -0.080968"
-      rpy="-1.5708 0 0" />
-    <parent
-      link="steer_front_right" />
-    <child
-      link="front_right_wheel" />
+      xyz="-0.000137084263775206 0.0908967088232522 -0.0809700175540105"
+      rpy="-1.5707963267949 0 0" />
+    <parent
+      link="steer_fl" />
+    <child
+      link="fl_wheel" />
     <axis
       xyz="0 0 -1" />
@@ -167,28 +282,27 @@
       velocity="100" />
   </joint>
-  <!-- Front Left Module -->
-  <link
-    name="steer_front_left">
-    <inertial>
-      <origin
-        xyz="0.000601677062523953 0.0211614748214363 -0.0742014114853441"
-        rpy="0 0 0" />
-      <mass
-        value="0.0538768857414007" />
-      <inertia
-        ixx="1.72828309289817E-05"
-        ixy="1.86491442781274E-10"
-        ixz="7.27396023667422E-08"
-        iyy="1.2650499347556E-05"
-        iyz="2.88105131447638E-12"
-        izz="1.01159127681761E-05" />
-    </inertial>
-    <visual>
-      <origin
-        xyz="0 0 0"
-        rpy="0 0 0" />
-      <geometry>
-        <mesh
-          filename="package://rocker_description/meshes/steer_front_left.STL" />
+  <link
+    name="steer_rl">
+    <inertial>
+      <origin
+        xyz="-0.000138607285511289 0.0211614748181154 -0.0742037209979592"
+        rpy="0 0 0" />
+      <mass
+        value="0.0538768866301723" />
+      <inertia
+        ixx="1.72835692098332E-05"
+        ixy="1.86529950289799E-10"
+        ixz="1.22949485862317E-09"
+        iyy="1.2650499668671E-05"
+        iyz="1.05181708221559E-12"
+        izz="1.01151748145831E-05" />
+    </inertial>
+    <visual>
+      <origin
+        xyz="0 0 0"
+        rpy="0 0 0" />
+      <geometry>
+        <mesh
+          filename="package://rocker_description/meshes/steer_rl.STL" />
       </geometry>
       <material
@@ -204,49 +318,49 @@
       <geometry>
         <mesh
-          filename="package://rocker_description/meshes/steer_front_left.STL" />
-      </geometry>
-    </collision>
-  </link>
-  <joint
-    name="steer_front_left_joint"
+          filename="package://rocker_description/meshes/steer_rl.STL" />
+      </geometry>
+    </collision>
+  </link>
+  <joint
+    name="steer_rl_joint"
     type="revolute">
     <origin
-      xyz="0.1075 0.16656 -0.028875"
-      rpy="0 0 0" />
-    <parent
-      link="base_link" />
-    <child
-      link="steer_front_left" />
-    <axis
-      xyz="0 0 -1" />
-    <limit
-      lower="-1.57"
-      upper="1.57"
-      effort="2"
-      velocity="3.14" />
-  </joint>
-  <link
-    name="front_left_wheel">
-    <inertial>
-      <origin
-        xyz="-1.47034815989322E-08 1.13284836511518E-08 -0.00840874583108248"
+      xyz="-0.109848463837903 0.036013571503488 0.0365656792825895"
+      rpy="1.5707963267949 0 0" />
+    <parent
+      link="T_left" />
+    <child
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
File: src/rocker_description/urdf/rocker_gazebo.xacro (robot description, xacro)
@@ -2,5 +2,5 @@
 <robot name="rocker" xmlns:xacro="http://ros.org/wiki/xacro">
   <!-- Wheels -->
-  <gazebo reference="front_left_wheel">
+  <gazebo reference="fl_wheel">
     <mu1>1.0</mu1>
     <mu2>1.0</mu2>
@@ -11,5 +11,5 @@
     <fdir1>1 0 0</fdir1>
   </gazebo>
-  <gazebo reference="rear_right_wheel">
+  <gazebo reference="rr_wheel">
     <mu1>1.0</mu1>
     <mu2>1.0</mu2>
@@ -20,5 +20,5 @@
     <fdir1>1 0 0</fdir1>
   </gazebo>
-  <gazebo reference="rear_left_wheel">
+  <gazebo reference="rl_wheel">
     <mu1>1.0</mu1>
     <mu2>1.0</mu2>
@@ -29,5 +29,5 @@
     <fdir1>1 0 0</fdir1>
   </gazebo>
-  <gazebo reference="front_right_wheel">
+  <gazebo reference="fr_wheel">
     <mu1>1.0</mu1>
     <mu2>1.0</mu2>
@@ -38,5 +38,5 @@
     <fdir1>1 0 0</fdir1>
   </gazebo>
-  <gazebo reference="steer_front_left">
+  <gazebo reference="steer_fl">
     <mu1>1.0</mu1>
     <mu2>1.0</mu2>
@@ -44,5 +44,5 @@
     <kd>10.0</kd>
   </gazebo>
-  <gazebo reference="steer_front_right">
+  <gazebo reference="steer_fr">
     <mu1>1.0</mu1>
     <mu2>1.0</mu2>
@@ -50,5 +50,5 @@
     <kd>10.0</kd>
   </gazebo>
-  <gazebo reference="steer_rear_left">
+  <gazebo reference="steer_rl">
     <mu1>1.0</mu1>
     <mu2>1.0</mu2>
@@ -56,5 +56,5 @@
     <kd>10.0</kd>
   </gazebo>
-  <gazebo reference="steer_rear_right">
+  <gazebo reference="steer_rr">
     <mu1>1.0</mu1>
     <mu2>1.0</mu2>

File: src/rocker_description/urdf/rocker_ros2_control.xacro (robot description, xacro)
@@ -11,5 +11,5 @@
     </xacro:if>
     <!-- DRIVE WHEEL JOINTS (VELOCITY CONTROL) -->
-    <joint name="front_right_wheel_joint">
+    <joint name="fr_wheel_joint">
       <command_interface name="velocity">
         <param name="min">-10</param>
@@ -19,5 +19,5 @@
       <state_interface name="velocity"/>
     </joint>
-    <joint name="front_left_wheel_joint">
+    <joint name="fl_wheel_joint">
       <command_interface name="velocity">
         <param name="min">-10</param>
@@ -27,5 +27,5 @@
       <state_interface name="velocity"/>
     </joint>
-    <joint name="rear_left_wheel_joint">
+    <joint name="rl_wheel_joint">
       <command_interface name="velocity">
         <param name="min">-10</param>
@@ -35,5 +35,5 @@
       <state_interface name="velocity"/>
     </joint>
-    <joint name="rear_right_wheel_joint">
+    <joint name="rr_wheel_joint">
       <command_interface name="velocity">
         <param name="min">-10</param>
@@ -44,20 +44,20 @@
     </joint>
     <!-- STEERING JOINTS (POSITION CONTROL) -->
-    <joint name="steer_front_left_joint">
+    <joint name="steer_fl_joint">
       <command_interface name="position"/>
       <state_interface name="position"/>
       <state_interface name="velocity"/>
     </joint>
-    <joint name="steer_front_right_joint">
+    <joint name="steer_fr_joint">
       <command_interface name="position"/>
       <state_interface name="position"/>
       <state_interface name="velocity"/>
     </joint>
-    <joint name="steer_rear_left_joint">
+    <joint name="steer_rl_joint">
       <command_interface name="position"/>
       <state_interface name="position"/>
       <state_interface name="velocity"/>
     </joint>
-    <joint name="steer_rear_right_joint">
+    <joint name="steer_rr_joint">
       <command_interface name="position"/>
       <state_interface name="position"/>
