Commit message: chassis isnt collapsing, not sure abt rocker

File: src/rocker_description/urdf/rocker.urdf.xacro (robot description, xacro)
@@ -14,15 +14,15 @@
     <inertial>
       <origin
-        xyz="-0.0029178 -1.0243E-05 0.026001"
-        rpy="0 0 0" />
-      <mass
-        value="3.0355" />
-      <inertia
-        ixx="0.011434"
-        ixy="8.2789E-18"
-        ixz="-1.2087E-05"
-        iyy="0.0094299"
-        iyz="-3.1877E-20"
-        izz="0.018372" />
+        xyz="0.00298859191128537 0.00327281389503588 0.0236277353082409"
+        rpy="0 0 0" />
+      <mass
+        value="3.54225026427668" />
+      <inertia
+        ixx="0.0133706956982974"
+        ixy="-2.17144708939564E-18"
+        ixz="-1.2927668928213E-05"
+        iyy="0.014433056958566"
+        iyz="-1.18489830462864E-19"
+        izz="0.0248980091378906" />
     </inertial>
     <visual>
@@ -51,18 +51,598 @@
   </link>
   <link
+    name="rocker_left">
+    <inertial>
+      <origin
+        xyz="-0.00596279660340987 0.019311656792217 0.00821775120018922"
+        rpy="0 0 0" />
+      <mass
+        value="0.548279466495107" />
+      <inertia
+        ixx="0.000160712183240721"
+        ixy="-1.18295175490068E-05"
+        ixz="4.65341036035169E-08"
+        iyy="0.00145712336713844"
+        iyz="2.38546497105557E-06"
+        izz="0.00150112676292675" />
+    </inertial>
+    <visual>
+      <origin
+        xyz="0 0 0"
+        rpy="0 0 0" />
+      <geometry>
+        <mesh
+          filename="package://rocker_description/meshes/rocker_left.STL" />
+      </geometry>
+      <material
+        name="">
+        <color
+          rgba="0.752941176470588 0.752941176470588 0.752941176470588 1" />
+      </material>
+    </visual>
+    <collision>
+      <origin
+        xyz="0 0 0"
+        rpy="0 0 0" />
+      <geometry>
+        <mesh
+          filename="package://rocker_description/meshes/rocker_left.STL" />
+      </geometry>
+    </collision>
+  </link>
+  <joint
+    name="rocker_left_joint"
+    type="revolute">
+    <origin
+      xyz="-0.012023 0.14327 0.0036435"
+      rpy="-1.5708 0 0" />
+    <parent
+      link="base_link" />
+    <child
+      link="rocker_left" />
+    <axis
+      xyz="0 0 -1" />
+    <limit
+      lower="-0.785"
+      upper="0.785"
+      effort="10"
+      velocity="20" />
+  </joint>
+  <link
+    name="steer_fl">
+    <inertial>
+      <origin
+        xyz="0.000519302806489791 0.00116147489574503 -0.072249011838569"
+        rpy="0 0 0" />
+      <mass
+        value="0.0538768873270146" />
+      <inertia
+        ixx="1.72835692633752E-05"
+        ixy="1.86524259779787E-10"
+        ixz="1.22947445955916E-09"
+        iyy="1.2650499733089E-05"
+        iyz="1.03479920307063E-12"
+        izz="1.0115174825469E-05" />
+    </inertial>
+    <visual>
+      <origin
+        xyz="0 0 0"
+        rpy="0 0 0" />
+      <geometry>
+        <mesh
+          filename="package://rocker_description/meshes/steer_fl.STL" />
+      </geometry>
+      <material
+        name="">
+        <color
+          rgba="0.752941176470588 0.752941176470588 0.752941176470588 1" />
+      </material>
+    </visual>
+    <collision>
+      <origin
+        xyz="0 0 0"
+        rpy="0 0 0" />
+      <geometry>
+        <mesh
+          filename="package://rocker_description/meshes/steer_fl.STL" />
+      </geometry>
+    </collision>
+  </link>
+  <joint
+    name="steer_fl_joint"
+    type="revolute">
+    <origin
+      xyz="0.10949 0.037941 0.046566"
+      rpy="1.5708 0 0" />
+    <parent
+      link="rocker_left" />
+    <child
+      link="steer_fl" />
+    <axis
+      xyz="0 0 -1" />
+    <limit
+      lower="-3.14"
+      upper="3.14"
+      effort="10"
+      velocity="20" />
+  </joint>
+  <link
+    name="fl_wheel">
+    <inertial>
+      <origin
+        xyz="0.00209895984803671 -0.00193945272577944 -0.0284087458310821"
+        rpy="0 0 0" />
+      <mass
+        value="0.13017290647518" />
+      <inertia
+        ixx="0.000124778074397082"
+        ixy="-7.56745189271209E-12"
+        ixz="-1.0927757268831E-11"
+        iyy="0.000124777976595369"
+        iyz="-2.36402552812522E-12"
+        izz="0.000234671292019043" />
+    </inertial>
+    <visual>
+      <origin
+        xyz="0 0 0"
+        rpy="0 0 0" />
+      <geometry>
+        <mesh
+          filename="package://rocker_description/meshes/fl_wheel.STL" />
+      </geometry>
+      <material
+        name="">
+        <color
+          rgba="0.792156862745098 0.819607843137255 0.933333333333333 1" />
+      </material>
+    </visual>
+    <collision>
+      <origin
+        xyz="0 0 0"
+        rpy="0 0 0" />
+      <geometry>
+        <mesh
+          filename="package://rocker_description/meshes/fl_wheel.STL" />
+      </geometry>
+    </collision>
+  </link>
+  <joint
+    name="fl_wheel_joint"
+    type="continuous">
+    <origin
+      xyz="-0.0015781 0.090897 -0.080955"
+      rpy="-1.5708 0 0" />
+    <parent
+      link="steer_fl" />
+    <child
+      link="fl_wheel" />
+    <axis
+      xyz="0 0 -1" />
+    <limit
+      lower="-10"
+      upper="10"
+      effort="10"
+      velocity="100" />
+  </joint>
+  <link
+    name="steer_rl">
+    <inertial>
+      <origin
+        xyz="0.000484941569044394 0.00116147486494461 -0.0761644406147317"
+        rpy="0 0 0" />
+      <mass
+        value="0.053876887039627" />
+      <inertia
+        ixx="1.72835692580122E-05"
+        ixy="1.86520191057722E-10"
+        ixz="1.22945286982952E-09"
+        iyy="1.26504997081888E-05"
+        iyz="1.03201975349867E-12"
+        izz="1.01151748056035E-05" />
+    </inertial>
+    <visual>
+      <origin
+        xyz="0 0 0"
+        rpy="0 0 0" />
+      <geometry>
+        <mesh
+          filename="package://rocker_description/meshes/steer_rl.STL" />
+      </geometry>
+      <material
+        name="">
+        <color
+          rgba="0.752941176470588 0.752941176470588 0.752941176470588 1" />
+      </material>
+    </visual>
+    <collision>
+      <origin
+        xyz="0 0 0"
+        rpy="0 0 0" />
+      <geometry>
+        <mesh
+          filename="package://rocker_description/meshes/steer_rl.STL" />
+      </geometry>
+    </collision>
+  </link>
+  <joint
+    name="steer_rl_joint"
+    type="revolute">
+    <origin
+      xyz="-0.11047 0.034053 0.046566"
+      rpy="1.5708 0 0" />
+    <parent
+      link="rocker_left" />
+    <child
+      link="steer_rl" />
+    <axis
+      xyz="0 0 -1" />
+    <limit
+      lower="-0.785"
+      upper="0.785"
+      effort="10"
+      velocity="20" />
+  </joint>
+  <link
+    name="rl_wheel">
+    <inertial>
+      <origin
+        xyz="0.00206456857074838 0.00197597049736126 -0.0284087458310854"
+        rpy="0 0 0" />
+      <mass
+        value="0.130172906475179" />
+      <inertia
+        ixx="0.000124777994283405"
+        ixy="3.83968738303507E-11"
+        ixz="1.71836065112964E-12"
+        iyy="0.000124778056709046"
+        iyz="1.10477040342025E-11"
+        izz="0.000234671292019043" />
+    </inertial>
+    <visual>
+      <origin
+        xyz="0 0 0"
+        rpy="0 0 0" />
+      <geometry>
+        <mesh
+          filename="package://rocker_description/meshes/rl_wheel.STL" />
+      </geometry>
+      <material
+        name="">
+        <color
+          rgba="0.792156862745098 0.819607843137255 0.933333333333333 1" />
+      </material>
+    </visual>
+    <collision>
+      <origin
+        xyz="0 0 0"
+        rpy="0 0 0" />
+      <geometry>
+        <mesh
+          filename="package://rocker_description/meshes/rl_wheel.STL" />
+      </geometry>
+    </collision>
+  </link>
+  <joint
+    name="rl_wheel_joint"
+    type="continuous">
+    <origin
+      xyz="-0.0015781 0.090897 -0.080955"
+      rpy="-1.5708 0 0" />
+    <parent
+      link="steer_rl" />
+    <child
+      link="rl_wheel" />
+    <axis
+      xyz="0 0 -1" />
+    <limit
+      lower="-10"
+      upper="10"
+      effort="10"
+      velocity="100" />
+  </joint>
+  <link
+    name="rocker_right">
+    <inertial>
+      <origin
+        xyz="-0.00596288573860194 -0.0193116567449316 0.00817977272543077"
+        rpy="0 0 0" />
+      <mass
+        value="0.548279467986759" />
+      <inertia
+        ixx="0.000160712214916101"
+        ixy="1.170043772776E-05"
+        ixz="-4.59530273941062E-08"
+        iyy="0.00145712333528538"
+        iyz="-2.31782015149321E-06"
+        izz="0.00150112676270733" />
+    </inertial>
+    <visual>
+      <origin
+        xyz="0 0 0"
+        rpy="0 0 0" />
+      <geometry>
+        <mesh
+          filename="package://rocker_description/meshes/rocker_right.STL" />
+      </geometry>
+      <material
+        name="">
+        <color
+          rgba="0.752941176470588 0.752941176470588 0.752941176470588 1" />
+      </material>
+    </visual>
+    <collision>
+      <origin
+        xyz="0 0 0"
+        rpy="0 0 0" />
+      <geometry>
+        <mesh
+          filename="package://rocker_description/meshes/rocker_right.STL" />
+      </geometry>
+    </collision>
+  </link>
+  <joint
+    name="rocker_right_joint"
+    type="revolute">
+    <origin
+      xyz="-0.012023 -0.13673 0.0036435"
+      rpy="1.5708 0 0" />
+    <parent
+      link="base_link" />
+    <child
+      link="rocker_right" />
+    <axis
+      xyz="0 0 -1" />
+    <limit
+      lower="-0.785"
+      upper="0.785"
+      effort="10"
+      velocity="100" />
+  </joint>
+  <link
+    name="steer_fr">
+    <inertial>
+      <origin
+        xyz="0.000814806413008712 -0.00116147492243543 -0.0722542108674373"
+        rpy="0 0 0" />
+      <mass
+        value="0.0538768878184284" />
+      <inertia
+        ixx="1.72835694548748E-05"
+        ixy="1.86529294081939E-10"
+        ixz="5.41767155045705E-10"
+        iyy="1.26504997493636E-05"
+        iyz="-9.96207531427938E-13"
+        izz="1.01151746557608E-05" />
+    </inertial>
+    <visual>
+      <origin
+        xyz="0 0 0"
+        rpy="0 0 0" />
+      <geometry>
+        <mesh
+          filename="package://rocker_description/meshes/steer_fr.STL" />
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
File: src/rocker_description/urdf/rocker_gazebo.xacro (robot description, xacro)
@@ -62,10 +62,32 @@
     <kd>10.0</kd>
   </gazebo>
-<gazebo>
-  <plugin filename="ign_ros2_control-system" name="ign_ros2_control::IgnitionROS2ControlPlugin">
-    <parameters>$(find rocker_controller)/config/rocker_controllers.yaml</parameters>
-  </plugin>
-  <plugin filename="ignition-gazebo-imu-system" name="ignition::gazebo::systems::Imu"/>
-  <plugin filename="ignition-gazebo-sensors-system" name="ignition::gazebo::systems::Sensors"/>
-</gazebo>
+  <gazebo>
+    <!-- ROS 2 Control Plugin -->
+    <plugin filename="ign_ros2_control-system" name="ign_ros2_control::IgnitionROS2ControlPlugin">
+      <parameters>$(find rocker_controller)/config/rocker_controllers.yaml</parameters>
+    </plugin>
+    <!-- IMU Sensor System -->
+    <!-- <plugin filename="ignition-gazebo-imu-system" name="ignition::gazebo::systems::Imu"/> -->
+    <!-- Sensor Management System -->
+    <!-- <plugin filename="ignition-gazebo-sensors-system" name="ignition::gazebo::systems::Sensors"/> -->
+    <!-- Detachable Joint Plugin to Simulate Multi-Parent (e.g., 4-bar style) -->
+    <plugin filename="libgz-sim-detachable-joint-system.so" name="gz::sim::systems::DetachableJoint">
+      <parent_link>rocker_left</parent_link>
+      <child_model>bot</child_model>
+      <child_link>diff_link</child_link>
+      <attach_topic>attach_diff_to_left</attach_topic>
+    </plugin>
+    <plugin filename="libgz-sim-detachable-joint-system.so" name="gz::sim::systems::DetachableJoint">
+      <parent_link>rocker_right</parent_link>
+      <child_model>bot</child_model>
+      <child_link>diff_link</child_link>
+      <attach_topic>attach_diff_to_right</attach_topic>
+    </plugin>
+    <!-- <plugin filename="libgz-sim-detachable-joint-system.so" name="gz::sim::systems::DetachableJoint">
+      <parent_link>base_link</parent_link>
+      <child_model>bot</child_model>
+      <child_link>diff_link</child_link>
+      <attach_topic>attach_diff_to_base</attach_topic>
+    </plugin> -->
+  </gazebo>
 </robot>
