Commit message: added connecting links

File: src/rocker_description/urdf/rocker.urdf.xacro (robot description, xacro)
@@ -14,15 +14,15 @@
     <inertial>
       <origin
-        xyz="0.00298859191128537 0.00327281389503588 0.0236277353082409"
-        rpy="0 0 0" />
-      <mass
-        value="3.54225026427668" />
-      <inertia
-        ixx="0.0133706956982974"
-        ixy="-2.17144708939564E-18"
-        ixz="-1.2927668928213E-05"
-        iyy="0.014433056958566"
-        iyz="-1.18489830462864E-19"
-        izz="0.0248980091378906" />
+        xyz="0.0036529 -1.0215E-05 0.02903"
+        rpy="0 0 0" />
+      <mass
+        value="3.2518" />
+      <inertia
+        ixx="0.012194"
+        ixy="-4.5489E-11"
+        ixz="-1.2673E-05"
+        iyy="0.0094514"
+        iyz="-9.282E-10"
+        izz="0.019133" />
     </inertial>
     <visual>
@@ -54,15 +54,15 @@
     <inertial>
       <origin
-        xyz="-0.00596279660340987 0.019311656792217 0.00821775120018922"
-        rpy="0 0 0" />
-      <mass
-        value="0.548279466495107" />
-      <inertia
-        ixx="0.000160712183240721"
-        ixy="-1.18295175490068E-05"
-        ixz="4.65341036035169E-08"
-        iyy="0.00145712336713844"
-        iyz="2.38546497105557E-06"
-        izz="0.00150112676292675" />
+        xyz="-0.0059628 0.019312 0.0082178"
+        rpy="0 0 0" />
+      <mass
+        value="0.54828" />
+      <inertia
+        ixx="0.00016071"
+        ixy="-1.183E-05"
+        ixz="4.6534E-08"
+        iyy="0.0014571"
+        iyz="2.3855E-06"
+        izz="0.0015011" />
     </inertial>
     <visual>
@@ -77,5 +77,5 @@
         name="">
         <color
-          rgba="0.752941176470588 0.752941176470588 0.752941176470588 1" />
+          rgba="0 0.4 0 1" />
       </material>
     </visual>
@@ -94,6 +94,6 @@
     type="revolute">
     <origin
-      xyz="-0.012023 0.14327 0.0036435"
-      rpy="-1.5708 0 0" />
+      xyz="-0.00300007366280326 0.139989762643875 0.00599815142431871"
+      rpy="-1.5707963267949 0 0" />
     <parent
       link="base_link" />
@@ -112,5 +112,5 @@
     <inertial>
       <origin
-        xyz="0.000519302806489791 0.00116147489574503 -0.072249011838569"
+        xyz="0.000519302806489763 0.00116147489574497 -0.072249011838569"
         rpy="0 0 0" />
       <mass
@@ -118,8 +118,8 @@
       <inertia
         ixx="1.72835692633752E-05"
-        ixy="1.86524259779787E-10"
-        ixz="1.22947445955916E-09"
+        ixy="1.86524259779789E-10"
+        ixz="1.22947445955912E-09"
         iyy="1.2650499733089E-05"
-        iyz="1.03479920307063E-12"
+        iyz="1.0347992030602E-12"
         izz="1.0115174825469E-05" />
     </inertial>
@@ -152,6 +152,6 @@
     type="revolute">
     <origin
-      xyz="0.10949 0.037941 0.046566"
-      rpy="1.5708 0 0" />
+      xyz="0.109493624388031 0.03794110103799 0.0465656792826112"
+      rpy="1.5707963267949 0 0" />
     <parent
       link="rocker_left" />
@@ -170,15 +170,15 @@
     <inertial>
       <origin
-        xyz="0.00209895984803671 -0.00193945272577944 -0.0284087458310821"
-        rpy="0 0 0" />
-      <mass
-        value="0.13017290647518" />
-      <inertia
-        ixx="0.000124778074397082"
-        ixy="-7.56745189271209E-12"
-        ixz="-1.0927757268831E-11"
-        iyy="0.000124777976595369"
-        iyz="-2.36402552812522E-12"
-        izz="0.000234671292019043" />
+        xyz="0.002099 -0.0019395 -0.028409"
+        rpy="0 0 0" />
+      <mass
+        value="0.13017" />
+      <inertia
+        ixx="0.00012478"
+        ixy="-7.5675E-12"
+        ixz="-1.0928E-11"
+        iyy="0.00012478"
+        iyz="-2.364E-12"
+        izz="0.00023467" />
     </inertial>
     <visual>
@@ -193,5 +193,5 @@
         name="">
         <color
-          rgba="0.792156862745098 0.819607843137255 0.933333333333333 1" />
+          rgba="0 0 0 1" />
       </material>
     </visual>
@@ -210,6 +210,6 @@
     type="continuous">
     <origin
-      xyz="-0.0015781 0.090897 -0.080955"
-      rpy="-1.5708 0 0" />
+      xyz="-0.0015781170593388 0.0908967088232542 -0.0809547532967621"
+      rpy="-1.5707963267949 0 0" />
     <parent
       link="steer_fl" />
@@ -228,5 +228,5 @@
     <inertial>
       <origin
-        xyz="0.000484941569044394 0.00116147486494461 -0.0761644406147317"
+        xyz="0.000484941569044396 0.00116147486494456 -0.0761644406147317"
         rpy="0 0 0" />
       <mass
@@ -234,8 +234,8 @@
       <inertia
         ixx="1.72835692580122E-05"
-        ixy="1.86520191057722E-10"
-        ixz="1.22945286982952E-09"
+        ixy="1.86520191057726E-10"
+        ixz="1.22945286982955E-09"
         iyy="1.26504997081888E-05"
-        iyz="1.03201975349867E-12"
+        iyz="1.03201975349808E-12"
         izz="1.01151748056035E-05" />
     </inertial>
@@ -268,10 +268,126 @@
     type="revolute">
     <origin
-      xyz="-0.11047 0.034053 0.046566"
-      rpy="1.5708 0 0" />
+      xyz="-0.110472012747799 0.0340528521482858 0.0465656792826093"
+      rpy="1.5707963267949 0 0" />
     <parent
       link="rocker_left" />
     <child
       link="steer_rl" />
+    <axis
+      xyz="0 0 -1" />
+    <limit
+      lower="-3.14"
+      upper="3.14"
+      effort="10"
+      velocity="20" />
+  </joint>
+  <link
+    name="rl_wheel">
+    <inertial>
+      <origin
+        xyz="0.0020646 0.001976 -0.028409"
+        rpy="0 0 0" />
+      <mass
+        value="0.13017" />
+      <inertia
+        ixx="0.00012478"
+        ixy="3.8397E-11"
+        ixz="1.7184E-12"
+        iyy="0.00012478"
+        iyz="1.1048E-11"
+        izz="0.00023467" />
+    </inertial>
+    <visual>
+      <origin
+        xyz="0 0 0"
+        rpy="0 0 0" />
+      <geometry>
+        <mesh
+          filename="package://rocker_description/meshes/rl_wheel.STL" />
+      </geometry>
+      <material
+        name="">
+        <color
+          rgba="0 0 0 1" />
+      </material>
+    </visual>
+    <collision>
+      <origin
+        xyz="0 0 0"
+        rpy="0 0 0" />
+      <geometry>
+        <mesh
+          filename="package://rocker_description/meshes/rl_wheel.STL" />
+      </geometry>
+    </collision>
+  </link>
+  <joint
+    name="rl_wheel_joint"
+    type="continuous">
+    <origin
+      xyz="-0.00157811705934295 0.0908967088232554 -0.0809547532967675"
+      rpy="-1.5707963267949 0 0" />
+    <parent
+      link="steer_rl" />
+    <child
+      link="rl_wheel" />
+    <axis
+      xyz="0 0 -1" />
+    <limit
+      lower="-10"
+      upper="10"
+      effort="10"
+      velocity="100" />
+  </joint>
+  <link
+    name="rocker_right">
+    <inertial>
+      <origin
+        xyz="-0.0059629 -0.019312 0.0081798"
+        rpy="0 0 0" />
+      <mass
+        value="0.54828" />
+      <inertia
+        ixx="0.00016071"
+        ixy="1.17E-05"
+        ixz="-4.5953E-08"
+        iyy="0.0014571"
+        iyz="-2.3178E-06"
+        izz="0.0015011" />
+    </inertial>
+    <visual>
+      <origin
+        xyz="0 0 0"
+        rpy="0 0 0" />
+      <geometry>
+        <mesh
+          filename="package://rocker_description/meshes/rocker_right.STL" />
+      </geometry>
+      <material
+        name="">
+        <color
+          rgba="0 0.4 0 1" />
+      </material>
+    </visual>
+    <collision>
+      <origin
+        xyz="0 0 0"
+        rpy="0 0 0" />
+      <geometry>
+        <mesh
+          filename="package://rocker_description/meshes/rocker_right.STL" />
+      </geometry>
+    </collision>
+  </link>
+  <joint
+    name="rocker_right_joint"
+    type="revolute">
+    <origin
+      xyz="-0.00300007366280228 -0.140010237356125 0.00599815142431871"
+      rpy="1.5707963267949 0 0" />
+    <parent
+      link="base_link" />
+    <child
+      link="rocker_right" />
     <axis
       xyz="0 0 -1" />
@@ -283,53 +399,111 @@
   </joint>
   <link
-    name="rl_wheel">
-    <inertial>
-      <origin
-        xyz="0.00206456857074838 0.00197597049736126 -0.0284087458310854"
-        rpy="0 0 0" />
-      <mass
-        value="0.130172906475179" />
-      <inertia
-        ixx="0.000124777994283405"
-        ixy="3.83968738303507E-11"
-        ixz="1.71836065112964E-12"
-        iyy="0.000124778056709046"
-        iyz="1.10477040342025E-11"
-        izz="0.000234671292019043" />
-    </inertial>
-    <visual>
-      <origin
-        xyz="0 0 0"
-        rpy="0 0 0" />
-      <geometry>
-        <mesh
-          filename="package://rocker_description/meshes/rl_wheel.STL" />
-      </geometry>
-      <material
-        name="">
-        <color
-          rgba="0.792156862745098 0.819607843137255 0.933333333333333 1" />
-      </material>
-    </visual>
-    <collision>
-      <origin
-        xyz="0 0 0"
-        rpy="0 0 0" />
-      <geometry>
-        <mesh
-          filename="package://rocker_description/meshes/rl_wheel.STL" />
-      </geometry>
-    </collision>
-  </link>
-  <joint
-    name="rl_wheel_joint"
+    name="steer_fr">
+    <inertial>
+      <origin
+        xyz="0.000814806464579348 -0.0011614749039093 -0.0722542108542284"
+        rpy="0 0 0" />
+      <mass
+        value="0.0538768875909339" />
+      <inertia
+        ixx="1.7283569439176E-05"
+        ixy="1.86519220841325E-10"
+        ixz="5.41777362598005E-10"
+        iyy="1.26504997368065E-05"
+        iyz="-9.95471491964069E-13"
+        izz="1.01151746572533E-05" />
+    </inertial>
+    <visual>
+      <origin
+        xyz="0 0 0"
+        rpy="0 0 0" />
+      <geometry>
+        <mesh
+          filename="package://rocker_description/meshes/steer_fr.STL" />
+      </geometry>
+      <material
+        name="">
+        <color
+          rgba="0.752941176470588 0.752941176470588 0.752941176470588 1" />
+      </material>
+    </visual>
+    <collision>
+      <origin
+        xyz="0 0 0"
+        rpy="0 0 0" />
+      <geometry>
+        <mesh
+          filename="package://rocker_description/meshes/steer_fr.STL" />
+      </geometry>
+    </collision>
+  </link>
+  <joint
+    name="steer_fr_joint"
+    type="revolute">
+    <origin
+      xyz="0.109199494929351 -0.0379359018234412 0.0464809030708809"
+      rpy="-1.5707963267949 0 0" />
+    <parent
+      link="rocker_right" />
+    <child
+      link="steer_fr" />
+    <axis
+      xyz="0 0 -1" />
+    <limit
+      lower="-3.14"
+      upper="3.14"
+      effort="10"
+      velocity="20" />
+  </joint>
+  <link
+    name="fr_wheel">
+    <inertial>
+      <origin
+        xyz="0.002099 -0.0019395 0.028409"
+        rpy="0 0 0" />
+      <mass
+        value="0.13017" />
+      <inertia
+        ixx="0.00012478"
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
File: src/rocker_description/urdf/rocker_gazebo.xacro (robot description, xacro)
@@ -68,12 +68,12 @@
     </plugin>
     <!-- IMU Sensor System -->
-    <!-- <plugin filename="ignition-gazebo-imu-system" name="ignition::gazebo::systems::Imu"/> -->
+    <plugin filename="ignition-gazebo-imu-system" name="ignition::gazebo::systems::Imu"/>
     <!-- Sensor Management System -->
-    <!-- <plugin filename="ignition-gazebo-sensors-system" name="ignition::gazebo::systems::Sensors"/> -->
+    <plugin filename="ignition-gazebo-sensors-system" name="ignition::gazebo::systems::Sensors"/>
     <!-- Detachable Joint Plugin to Simulate Multi-Parent (e.g., 4-bar style) -->
     <plugin filename="libgz-sim-detachable-joint-system.so" name="gz::sim::systems::DetachableJoint">
       <parent_link>rocker_left</parent_link>
       <child_model>bot</child_model>
-      <child_link>diff_link</child_link>
+      <child_link>clink_left</child_link>
       <attach_topic>attach_diff_to_left</attach_topic>
     </plugin>
@@ -81,5 +81,5 @@
       <parent_link>rocker_right</parent_link>
       <child_model>bot</child_model>
-      <child_link>diff_link</child_link>
+      <child_link>clink_right</child_link>
       <attach_topic>attach_diff_to_right</attach_topic>
     </plugin>
